Commit message: Modified ndt_matching to publish /estimated_vel and /time_ndt_matching.

File: ros/src/computing/perception/localization/packages/ndt_localizer/urdf/prius_model.urdf (robot description, URDF)
Before this commit: robot prius, 1 links, 0 joints
Links:
- link velodyne: geometry visual mesh filename=package://ndt_localizer/urdf/prius_model.dae scale=1.0 1.0 1.0
