Commit message: Tuned gazebo parameter

File: ros/src/system/gazebo/catvehicle/urdf/catvehicle.xacro (robot description, xacro)
@@ -102,10 +102,10 @@
       <parent link="base_link"/>
       <child link="main_mass"/>
-      <origin xyz="0 0 0" rpy="0 0 0"/>
+      <origin xyz="${tyre_x} 0 ${base_height}" rpy="0 0 0"/>
 </joint>
 <link name="main_mass" type="fixed">
      <parent link="inertial_joint"/>
      <inertial>
-        <origin xyz="${tyre_x} 0 ${base_height}" rpy="0 0 0"/>
+        <origin xyz="0 0 0" rpy="0 0 0"/>
         <mass value="${base_mass}"/>
         <inertia
