Commit message: move urdf and dae files

File: ros/src/vehicle/vehicle_description/urdf/default.urdf (robot description, URDF)
Before this commit: robot car, 1 links, 0 joints
Links:
- link base_link: geometry visual mesh filename=package://vehicle_description/mesh/CAR_original.dae scale=1.0 1.0 1.0

File: ros/src/vehicle/vehicle_description/urdf/estima_black.urdf (robot description, URDF)
Before this commit: robot car, 1 links, 0 joints
Links:
- link base_link: geometry visual mesh filename=package://vehicle_description/mesh/estima_black.dae scale=1.0 1.0 1.0

File: ros/src/vehicle/vehicle_description/urdf/estima_gray.urdf (robot description, URDF)
Before this commit: robot car, 1 links, 0 joints
Links:
- link base_link: geometry visual mesh filename=package://vehicle_description/mesh/estima_gray.dae scale=1.0 1.0 1.0

File: ros/src/vehicle/vehicle_description/urdf/estima_white.urdf (robot description, URDF)
Before this commit: robot car, 1 links, 0 joints
Links:
- removed link sim_base_link
- added link base_link; visual mesh filename=package://vehicle_description/mesh/estima_white.dae scale=1.0 1.0 1.0

File: ros/src/vehicle/vehicle_description/urdf/milee.urdf (robot description, URDF)
Before this commit: robot car, 1 links, 0 joints
Links:
- link base_link: geometry visual mesh filename=package://vehicle_description/mesh/milee.dae scale=1.5 1.5 1.5

File: ros/src/vehicle/vehicle_description/urdf/prius.urdf (robot description, URDF)
Before this commit: robot car, 1 links, 0 joints
Links:
- link base_link: geometry visual mesh filename=package://vehicle_description/mesh/prius.dae scale=1.0 1.0 1.0

File: ros/src/vehicle/vehicle_description/urdf/sim_default.urdf (robot description, URDF)
Before this commit: robot car, 1 links, 0 joints
Links:
- removed link base_link
- added link sim_base_link; visual mesh filename=package://vehicle_description/mesh/CAR_original.dae scale=1.0 1.0 1.0
